File: temp_probe_zigbee/temp_probe_zigbee.kicad_sch (KiCad schematic)
At the start: 0 parts

Commit message: Update KiCad design; ignore KiCad/JLCPCB local artifacts
Commit the latest schematic/PCB/project edits. Ignore regenerable artifacts:
auto-backups, *.kicad_prl, jlcpcb/ fab output, and stray *.rpt reports.

Co-Authored-By: Claude Opus 4.8 <noreply@anthropic.com>
Claude-Session: https://claude.ai/code/session_01PDqNxEFAhmrqW476w8fymk
Parts:
- added J1: Conn_01x08, Connector_PinSocket_2.54mm:PinSocket_1x08_P2.54mm_Vertical, symbol Connector_Generic:Conn_01x08
- added U1: XIAO-ESP32-C6, Seeed Studio XIAO Series Library:XIAO-ESP32C6-DIP, symbol Seeed_Studio_XIAO_Series:XIAO_ESP32-C6-DIP
Connections:
- new net +3.3V: J1.3 (Pin_3), U1.12 (3V3)
- new net CLK: J1.4 (Pin_4), U1.9 (GPIO19/D8/SCK)
- new net CS: J1.7 (Pin_7), U1.6 (GPIO23/D5/SCL)
- new net GND: J1.2 (Pin_2), U1.13 (GND)
- new net RDY: J1.8 (Pin_8), U1.5 (GPIO22/D4/SDA)
- new net SDI: J1.6 (Pin_6), U1.11 (GPIO18/D10/MOSI)
- new net SDO: J1.5 (Pin_5), U1.10 (GPIO20/D9/MISO)
- new net VIN: J1.1 (Pin_1)
- no-connect marks 0 -> 8
